Commit message: 0712

File: src/ur5/ur5_description/urdf/hand_rail.xacro (robot description, xacro)
@@ -7,5 +7,5 @@
         <parent link="${connected_to}"/>
         <child link="${ns}_hand"/>
-        <origin xyz="${xyz}" rpy="${rpy}"/>
+        <origin xyz="${xyz}" rpy="0 0 ${pi/2}"/>
       </joint>
     </xacro:unless>

File: src/ur5/ur5_description/urdf/ur5.urdf.xacro (robot description, xacro)
@@ -314,5 +314,5 @@
       <parent link="${prefix}wrist_3_link" />
       <child link = "${prefix}ee_link" />
-      <origin xyz="0.0 ${wrist_3_length} 0.0" rpy="0.0 0.0 ${pi/2.0}" />
+      <origin rpy="${-pi/2} 0 0" xyz="0 0.16 0"/>
     </joint>
     <link name="${prefix}ee_link">
