Commit message: 0904

File: src/ur5/ur5_description/urdf/kitchen.xacro (robot description, xacro)
@@ -3,5 +3,5 @@
     <!-- table -->
     <xacro:property name="table_w" value="0.5"/>
-    <xacro:property name="table_l" value="3.0"/>
+    <xacro:property name="table_l" value="3.45"/>
     <xacro:property name="table_h" value="0.4"/>
     <xacro:property name="table_dx" value="0.5"/>
@@ -31,5 +31,5 @@
     <!-- sauce shelf -->
     <xacro:property name="shelf_w" value="0.2"/>
-    <xacro:property name="shelf_l" value="0.8"/>
+    <xacro:property name="shelf_l" value="1.0"/>
     <xacro:property name="shelf_h" value="0.02"/>
     <xacro:property name="shelf_dh" value="0.1"/>

File: src/ur5/ur5_description/urdf/ur5.urdf.xacro (robot description, xacro)
@@ -88,5 +88,5 @@
       <parent link="${prefix}rail0"/>
       <child link="${prefix}rail1"/>
-      <origin xyz="0 0 0.07" rpy="0 0 0"/>
+      <origin xyz="0 0 0.06" rpy="0 0 0"/>
       <axis xyz="0 1 0"/>
       <limit effort="30" velocity="1.0" lower="-2" upper="2"/>
@@ -315,5 +315,5 @@
       <parent link="${prefix}wrist_3_link" />
       <child link = "${prefix}ee_link" />
-      <origin rpy="${-pi/2} 0 0" xyz="0 0.1787
+      <origin rpy="${-pi/2} 0 0" xyz="0 0.175
        0"/>
     </joint>
