Commit message: 0713

File: src/ur5/ur5_description/urdf/ur5.urdf.xacro (robot description, xacro)
@@ -314,5 +314,5 @@
       <parent link="${prefix}wrist_3_link" />
       <child link = "${prefix}ee_link" />
-      <origin rpy="${-pi/2} 0 0" xyz="0 0.16 0"/>
+      <origin rpy="${-pi/2} 0 0" xyz="0 0.145 0"/>
     </joint>
     <link name="${prefix}ee_link">

Commit message: first commit

File: src/ur5/ur5_description/urdf/ur5.urdf.xacro (robot description, xacro)
@@ -72,5 +72,5 @@
       <visual>
         <geometry>
-          <box size="0.1 0.1 0.01"/>
+          <box size="0.1 0.1 0.1"/>
           <!-- <box size="1 1 1"/> -->
         </geometry>
@@ -81,4 +81,5 @@
     </link>
     <joint name="world_joint" type="fixed">
+        <origin xyz="0 0 0.05" rpy="0 0 0"/>
         <parent link="world"/>
         <child link="${prefix}rail0"/>
@@ -87,5 +88,5 @@
       <parent link="${prefix}rail0"/>
       <child link="${prefix}rail1"/>
-      <origin xyz="0 0 0" rpy="0 0 0"/>
+      <origin xyz="0 0 0.05" rpy="0 0 0"/>
       <axis xyz="0 1 0"/>
       <limit effort="30" velocity="1.0" lower="-2" upper="2"/>

Commit message: 0714

File: src/ur5/ur5_description/urdf/ur5.urdf.xacro (robot description, xacro)
@@ -345,4 +345,32 @@
       <child link="${prefix}tool0"/>
     </joint>
+    <link name="${prefix}_link_knife"/>
+    <joint name="${prefix}_joint_knife" type="fixed">
+        <origin rpy="0 0 0" xyz="0 0.21 0.039"/>
+        <!-- <origin rpy="0 0 0" xyz="0 0.21 0.019"/> -->
+        <parent link="${prefix}ee_link"/>
+        <child link="${prefix}_link_knife"/>
+    </joint>
+    <link name="${prefix}_link_spatula"/>
+    <joint name="${prefix}_joint_spatula" type="fixed">
+        <origin rpy="0 0 0" xyz="0 0.235 0"/>
+        <!-- <origin rpy="0 0 0" xyz="0 0.235 -0.02"/> -->
+        <parent link="${prefix}ee_link"/>
+        <child link="${prefix}_link_spatula"/>
+    </joint>
+    <link name="${prefix}_link_scooper"/>
+    <joint name="${prefix}_joint_scooper" type="fixed">
+        <origin rpy="0 0 0" xyz="0 0.25 0"/>
+        <!-- <origin rpy="0 0 0" xyz="0 0.25 -0.02"/> -->
+        <parent link="${prefix}ee_link"/>
+        <child link="${prefix}_link_scooper"/>
+    </joint>
+    <link name="${prefix}_link_spreader"/>
+    <joint name="${prefix}_joint_spreader" type="fixed">
+        <origin rpy="0 0 0" xyz="0 0.295 -0.002"/>
+        <!-- <origin rpy="0 0 0" xyz="0 0.295 -0.022"/> -->
+        <parent link="${prefix}ee_link"/>
+        <child link="${prefix}_link_spreader"/>
+    </joint>
   </xacro:macro>
 </robot>

Commit message: 0715

File: src/ur5/ur5_description/urdf/ur5.urdf.xacro (robot description, xacro)
@@ -315,5 +315,5 @@
       <parent link="${prefix}wrist_3_link" />
       <child link = "${prefix}ee_link" />
-      <origin rpy="${-pi/2} 0 0" xyz="0 0.145 0"/>
+      <origin rpy="${-pi/2} 0 0" xyz="0 0.135 0"/>
     </joint>
     <link name="${prefix}ee_link">

Commit message: 0718

File: src/ur5/ur5_description/urdf/ur5.urdf.xacro (robot description, xacro)
@@ -72,5 +72,5 @@
       <visual>
         <geometry>
-          <box size="0.1 0.1 0.1"/>
+          <box size="0.1 0.1 0.01"/>
           <!-- <box size="1 1 1"/> -->
         </geometry>
@@ -81,5 +81,5 @@
     </link>
     <joint name="world_joint" type="fixed">
-        <origin xyz="0 0 0.05" rpy="0 0 0"/>
+        <!-- <origin xyz="0 0 0.025" rpy="0 0 0"/> -->
         <parent link="world"/>
         <child link="${prefix}rail0"/>
@@ -88,5 +88,5 @@
       <parent link="${prefix}rail0"/>
       <child link="${prefix}rail1"/>
-      <origin xyz="0 0 0.05" rpy="0 0 0"/>
+      <origin xyz="0 0 0.08" rpy="0 0 0"/>
       <axis xyz="0 1 0"/>
       <limit effort="30" velocity="1.0" lower="-2" upper="2"/>
@@ -315,5 +315,5 @@
       <parent link="${prefix}wrist_3_link" />
       <child link = "${prefix}ee_link" />
-      <origin rpy="${-pi/2} 0 0" xyz="0 0.135 0"/>
+      <origin rpy="${-pi/2} 0 0" xyz="0 0.165 0"/>
     </joint>
     <link name="${prefix}ee_link">

File: src/ur5/ur5_description/urdf/ur5_panda_rail.urdf (robot description, URDF)
Before this commit: robot ur5, 11 links, 10 joints
Links:
- added link _link_knife
- added link _link_scooper
- added link _link_spatula
- added link _link_spreader
- added link panda_hand; collision cylinder length=0.1 radius=0.04; collision sphere radius=0.01
- added link panda_leftfinger; visual mesh filename=package://franka_description/meshes/visual/finger.dae
- added link panda_rightfinger; visual mesh filename=package://franka_description/meshes/visual/finger.dae
- added link rail0; visual box size=0.1 0.1 0.01
- added link rail1; visual box size=0.1 0.1 0.01
Joints:
- added joint _joint_knife: type fixed, parent ee_link, child _link_knife, origin xyz=0 0.21 0.039 rpy=0 0 0
- added joint _joint_scooper: type fixed, parent ee_link, child _link_scooper, origin xyz=0 0.25 0 rpy=0 0 0
- added joint _joint_spatula: type fixed, parent ee_link, child _link_spatula, origin xyz=0 0.235 0 rpy=0 0 0
- added joint _joint_spreader: type fixed, parent ee_link, child _link_spreader, origin xyz=0 0.295 -0.002 rpy=0 0 0
- added joint base_joint: type fixed, parent rail1, child base_link
- added joint panda_finger_joint1: type prismatic, parent panda_hand, child panda_leftfinger, origin xyz=0 0 0.0584 rpy=0 0 0, axis 0 1 0, limit lower=0.0 upper=0.04 effort=20 velocity=0.2
- added joint panda_finger_joint2: type prismatic, parent panda_hand, child panda_rightfinger, origin xyz=0 0 0.0584 rpy=0 0 0, axis 0 -1 0, limit lower=0.0 upper=0.04 effort=20 velocity=0.2, mimic joint=panda_finger_joint1
- added joint panda_hand_joint: type fixed, parent tool0, child panda_hand, origin xyz=0 0 0 rpy=0 0 1.57079632679
- added joint rail_joint: type prismatic, parent rail0, child rail1, origin xyz=0 0 0.08 rpy=0 0 0, axis 0 1 0, limit lower=-2 upper=2 effort=30 velocity=1.0
- joint ee_fixed_joint: origin xyz=0.0 0.0823 0.0 rpy=0.0 0.0 1.57079632679 -> xyz=0 0.165 0 rpy=-1.57079632679 0 0
- joint world_joint: child base_link -> rail0; origin xyz=0.0 0.0 0.0 rpy=0.0 0.0 0.0 -> (none)

Commit message: 0721

File: src/ur5/ur5_description/urdf/ur5.urdf.xacro (robot description, xacro)
@@ -315,5 +315,5 @@
       <parent link="${prefix}wrist_3_link" />
       <child link = "${prefix}ee_link" />
-      <origin rpy="${-pi/2} 0 0" xyz="0 0.165 0"/>
+      <origin rpy="${-pi/2} 0 0" xyz="0 0.169 0"/>
     </joint>
     <link name="${prefix}ee_link">

Commit message: 0726

File: src/ur5/ur5_description/urdf/ur5.urdf.xacro (robot description, xacro)
@@ -315,5 +315,5 @@
       <parent link="${prefix}wrist_3_link" />
       <child link = "${prefix}ee_link" />
-      <origin rpy="${-pi/2} 0 0" xyz="0 0.169 0"/>
+      <origin rpy="${-pi/2} 0 0" xyz="0 0.175 0"/>
     </joint>
     <link name="${prefix}ee_link">

Commit message: 0727

File: src/ur5/ur5_description/urdf/ur5.urdf.xacro (robot description, xacro)
@@ -315,5 +315,5 @@
       <parent link="${prefix}wrist_3_link" />
       <child link = "${prefix}ee_link" />
-      <origin rpy="${-pi/2} 0 0" xyz="0 0.175 0"/>
+      <origin rpy="${-pi/2} 0 0" xyz="0 0.173 0"/>
     </joint>
     <link name="${prefix}ee_link">

Commit message: 0729

File: src/ur5/ur5_description/urdf/ur5.urdf.xacro (robot description, xacro)
@@ -315,5 +315,5 @@
       <parent link="${prefix}wrist_3_link" />
       <child link = "${prefix}ee_link" />
-      <origin rpy="${-pi/2} 0 0" xyz="0 0.173 0"/>
+      <origin rpy="${-pi/2} 0 0" xyz="0 0.18 0"/>
     </joint>
     <link name="${prefix}ee_link">

Commit message: 0808

File: src/ur5/ur5_description/urdf/ur5.urdf.xacro (robot description, xacro)
@@ -315,5 +315,5 @@
       <parent link="${prefix}wrist_3_link" />
       <child link = "${prefix}ee_link" />
-      <origin rpy="${-pi/2} 0 0" xyz="0 0.18 0"/>
+      <origin rpy="${-pi/2} 0 0" xyz="0 0.175 0"/>
     </joint>
     <link name="${prefix}ee_link">

Commit message: 0820

File: src/ur5/ur5_description/urdf/ur5.urdf.xacro (robot description, xacro)
@@ -88,5 +88,5 @@
       <parent link="${prefix}rail0"/>
       <child link="${prefix}rail1"/>
-      <origin xyz="0 0 0.07" rpy="0 0 0"/>
+      <origin xyz="0 0 0.06" rpy="0 0 0"/>
       <axis xyz="0 1 0"/>
       <limit effort="30" velocity="1.0" lower="-2" upper="2"/>
@@ -315,5 +315,5 @@
       <parent link="${prefix}wrist_3_link" />
       <child link = "${prefix}ee_link" />
-      <origin rpy="${-pi/2} 0 0" xyz="0 0.1787
+      <origin rpy="${-pi/2} 0 0" xyz="0 0.175
        0"/>
     </joint>

Commit message: 0824

File: src/ur5/ur5_description/urdf/ur5.urdf.xacro (robot description, xacro)
@@ -88,5 +88,5 @@
       <parent link="${prefix}rail0"/>
       <child link="${prefix}rail1"/>
-      <origin xyz="0 0 0.06" rpy="0 0 0"/>
+      <origin xyz="0 0 0.07" rpy="0 0 0"/>
       <axis xyz="0 1 0"/>
       <limit effort="30" velocity="1.0" lower="-2" upper="2"/>
@@ -315,5 +315,5 @@
       <parent link="${prefix}wrist_3_link" />
       <child link = "${prefix}ee_link" />
-      <origin rpy="${-pi/2} 0 0" xyz="0 0.175
+      <origin rpy="${-pi/2} 0 0" xyz="0 0.1787
        0"/>
     </joint>

Commit message: 0912

File: src/ur5/ur5_description/urdf/ur5.urdf.xacro (robot description, xacro)
@@ -88,5 +88,5 @@
       <parent link="${prefix}rail0"/>
       <child link="${prefix}rail1"/>
-      <origin xyz="0 0 0.06" rpy="0 0 0"/>
+      <origin xyz="0 0 0.08" rpy="0 0 0"/>
       <axis xyz="0 1 0"/>
       <limit effort="30" velocity="1.0" lower="-2" upper="2"/>

Commit message: 0914

File: src/ur5/ur5_description/urdf/ur5.urdf.xacro (robot description, xacro)
@@ -88,5 +88,5 @@
       <parent link="${prefix}rail0"/>
       <child link="${prefix}rail1"/>
-      <origin xyz="0 0 0.08" rpy="0 0 0"/>
+      <origin xyz="0 0 0.07" rpy="0 0 0"/>
       <axis xyz="0 1 0"/>
       <limit effort="30" velocity="1.0" lower="-2" upper="2"/>
@@ -315,5 +315,5 @@
       <parent link="${prefix}wrist_3_link" />
       <child link = "${prefix}ee_link" />
-      <origin rpy="${-pi/2} 0 0" xyz="0 0.175
+      <origin rpy="${-pi/2} 0 0" xyz="0 0.1787
        0"/>
     </joint>
