Commit message: 0809

File: src/franka_description/robots/panda_arm_hand.urdf_rail.xacro (robot description, xacro)
@@ -5,5 +5,6 @@
     <xacro:panda_arm connected_to="world" safety_distance="0.005"/>
     <xacro:hand ns="panda" rpy="0 0 ${-pi/4}" connected_to="panda_link8" safety_distance="0.00"/>
-    <!-- table -->
+</robot>
+    <!-- table
     <xacro:property name="table_w" value="0.5"/>
     <xacro:property name="table_l" value="3.0"/>
@@ -116,4 +117,3 @@
             </geometry>
         </collision>
-    </link>
-</robot>
+    </link> -->

File: src/ur5/ur5_description/urdf/ur5.urdf.xacro (robot description, xacro)
@@ -88,5 +88,5 @@
       <parent link="${prefix}rail0"/>
       <child link="${prefix}rail1"/>
-      <origin xyz="0 0 0.08" rpy="0 0 0"/>
+      <origin xyz="0 0 0.07" rpy="0 0 0"/>
       <axis xyz="0 1 0"/>
       <limit effort="30" velocity="1.0" lower="-2" upper="2"/>
@@ -315,5 +315,6 @@
       <parent link="${prefix}wrist_3_link" />
       <child link = "${prefix}ee_link" />
-      <origin rpy="${-pi/2} 0 0" xyz="0 0.175 0"/>
+      <origin rpy="${-pi/2} 0 0" xyz="0 0.1787
+       0"/>
     </joint>
     <link name="${prefix}ee_link">
